Commit message: Dispose to enable swapping models; fix stl

File: test/testdata/basic_with_stl_mesh.urdf (robot description, URDF)
Before this commit: robot myfirst, 1 links, 0 joints
Links:
- link base_link: geometry visual mesh filename=https://c%2B.vscode-resource.vscode-cdn.net/%5Cws%5Cjetbot%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

Commit message: Use Embedded Textures instead of forcing

File: test/testdata/basic_with_stl_mesh.urdf (robot description, URDF)
Before this commit: robot myfirst, 1 links, 0 joints
Links:
- link base_link: geometry visual mesh filename=file://../test/testdata/xyz_cube.stl

Commit message: Finish handling complex dae

File: test/testdata/basic_with_stl_mesh.urdf (robot description, URDF)
Before this commit: robot myfirst, 1 links, 0 joints
Links:
- link base_link: geometry visual mesh filename=https://raw.githubusercontent.com/polyhobbyist/babylon_ros/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

Commit message: Add test selection list

File: test/testdata/basic_with_stl_mesh.urdf (robot description, URDF)
Before this commit: robot myfirst, 1 links, 0 joints
Links:
- link base_link: geometry visual mesh filename=https://github.com/polyhobbyist/babylon_ros/blob/5d3fad9df8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

Commit message: Fix url basic_with_stl_mesh.urdf

File: test/testdata/basic_with_stl_mesh.urdf (robot description, URDF)
Before this commit: robot myfirst, 1 links, 0 joints
Links:
- link base_link: geometry visual mesh filename=https://github.com/polyhobbyist/babylon_ros/raw/5d3fad9df86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
