Commit message: feat: Update package configuration and module imports
- Added "type": "module" to package.json for ES module support.
- Updated "exports" field in package.json to specify import and types paths.
- Changed Babylon.js dependencies from version 8.0.x to 8.1.x.
- Updated devDependencies including typescript and ts-jest versions.
- Modified import statements in various source files to include ".js" extensions.
- Enhanced RobotScene class with improved hand tracking features and logging.
- Updated viewer.html to use ES module imports for Babylon.js.
- Refactored webpack configuration to support ESM output and module format.
- Adjusted test files to reflect changes in import paths.

File: test/testdata/basic_with_joint_with_effort.urdf (robot description, URDF)
Before this commit: robot origins, 2 links, 1 joints
Joints:
- joint base_to_right_leg: limit lower=0 upper=10 effort=1.1369 velocity=4.36 -> lower=-1 upper=1 effort=1.1369 velocity=4.36
