Commit message: fix: Update file paths in launch.json and adjust scaling in GeometryMesh; bump version to 0.1.4

File: test/testdata/bb.urdf (robot description, URDF)
Before this commit: robot bb_head, 6 links, 5 joints
Links:
- link base_link: geometry visual mesh filename=https://raw.githubusercontent.com/polyhobbyist/bb_descripti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 scale=0.00001 0.00001 0.00001
