Commit message: Update mule.urdf

File: test/testdata/mule.urdf (robot description, URDF)
Before this commit: robot mule, 7 links, 6 joints
Links:
- link left_front_wheel_link: geometry collision cylinder length=0.0889 radius=0.127; visual mesh filename=https://raw.githubusercontent.com/polyhobbyist/babylon_ros/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
- link left_mid_wheel_link: geometry collision cylinder length=0.0889 radius=0.127; visual mesh filename=https://raw.githubusercontent.com/polyhobbyist/babylon_ros/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
- link left_rear_wheel_link: geometry collision cylinder length=0.0889 radius=0.127; visual mesh filename=https://raw.githubusercontent.com/polyhobbyist/babylon_ros/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
- link right_front_wheel_link: geometry collision cylinder length=0.0889 radius=0.127; visual mesh filename=https://raw.githubusercontent.com/polyhobbyist/babylon_ros/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
- link right_mid_wheel_link: geometry collision cylinder length=0.0889 radius=0.127; visual mesh filename=https://raw.githubusercontent.com/polyhobbyist/babylon_ros/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
- link right_rear_wheel_link: geometry collision cylinder length=0.0889 radius=0.127; visual mesh filename=https://raw.githubusercontent.com/polyhobbyist/babylon_ros/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

Commit message: Fix mule

File: test/testdata/mule.urdf (robot description, URDF)
Before this commit: robot mule, 7 links, 6 joints
Joints:
- joint left_front_wheel: axis 0 1 0 -> 1 0 0
- joint left_mid_wheel: axis 0 1 0 -> 1 0 0
- joint left_rear_wheel: axis 0 1 0 -> 1 0 0
- joint right_front_wheel: axis 0 1 0 -> 1 0 0
- joint right_mid_wheel: axis 0 1 0 -> 1 0 0
- joint right_rear_wheel: axis 0 1 0 -> 1 0 0
